Commit message: 添加工具文件

File: src/agv_description/urdf/agv.xacro (robot description, xacro)
@@ -947,6 +947,17 @@
     <limit effort = "1000.0" velocity = "1.0" lower = "-3.0" upper = "3.0"/>
   </joint>
-  <link
-    name="arm2_tool_link" />
+ <link
+    name="arm2_tool_link" >
+  <visual>
+      <origin
+        xyz="0 0.145 -0.0748"
+        rpy="0 0 3.14159" />
+      <geometry>
+          <mesh
+    filename="package://agv_description/meshes/tool.STL"
+    scale="0.001 0.001 0.001" />
+      </geometry>
+    </visual>
+  </link>
   <joint
     name="arm2_tool_joint" type="fixed">
@@ -961,5 +972,5 @@
       <parent link="arm2_tool_link" />
       <child link="arm2_toolscan_link" />
-      <origin xyz="0 0.20 0" rpy="-1.5708 0 0" />
+      <origin xyz="0 0.145 0" rpy="-1.5708 0 0" />
   </joint>
 </robot>
